File: Projects/BeagleBone-Black-Cape/BeagleBone-Black-Cape.kicad_pcb (KiCad board)
At the start: 2 copper layers, 86.4 x 54.6 mm, 6 parts, among them P8 BeagleBone_Black_Header, P9 BeagleBone_Black_Header

Commit message: feat: update kicad-templates to 9.0.0-1
Signed-off-by: lhdjply <lhdjply@126.com>
Connections:
- P8 pad 26: /GPIO61 -> /LCD.PCLK
- P8 pad 28: /LCD.PCLK -> /GPIO61
