File: Projects/Edgeberry_Cartridge/Edgeberry_cartridge_template.kicad_pcb (KiCad board)
At the start: 2 copper layers, 49.8 x 63.2 mm, 1 part

Commit message: feat: update kicad-templates to 9.0.0-1
Signed-off-by: lhdjply <lhdjply@126.com>
Connections:
- H1 pad 2: Net-(H1-GPIO_21) -> unconnected-(H1-GPIO_21-Pad2)
