File: Projects/Edgeberry_Cartridge/Edgeberry_cartridge_template.kicad_sch (KiCad schematic)
At the start: 1 part

Commit message: feat: update kicad-templates to 9.0.0-1
Signed-off-by: lhdjply <lhdjply@126.com>
Changed lines of the file:
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@@
 (kicad_sch
-	(version 20231120)
+	(version 20250114)
 	(generator "eeschema")
-	(generator_version "8.0")
+	(generator_version "9.0")
 	(paper "A4")
 	(symbol
@@
 		)
 	)
+	(embedded_fonts no)
 )
