File: Projects/RaspberryPi-uHAT/RaspberryPi-uHAT.kicad_sch (KiCad schematic)
At the start: 6 parts, among them J1 GPIO, U1 CAT24C256

Commit message: feat: update kicad-templates to 9.0.0-1
Signed-off-by: lhdjply <lhdjply@126.com>
Changed lines of the file:
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@@
 (kicad_sch
-	(version 20231120)
+	(version 20250114)
 	(generator "eeschema")
-	(generator_version "8.0")
+	(generator_version "9.0")
 	(paper "A4")
 	(title_block
 		(date "15 nov 2012")
+	)
+	(text "ID_SD and ID_SC PINS:\nThese pins are reserved for HAT ID EEPROM.\n\nAt boot time this I2C interface will be\ninterrogated to look for an EEPROM\nthat identifes the attached board and\nallows automagic setup of the GPIOs\n(and optionally, Linux drivers).\n\nBridging JP1 enables write protection.\n\nDO NOT USE these pins for anything other\nthan attaching an I2C ID EEPROM. Leave\nunconnected if ID EEPROM not required."
+		(exclude_from_sim no)
+		(at 16.51 193.04 0)
+		(effects
+			(font
+				(size 1.27 1.27)
+			)
+			(justify left bottom)
+		)
+	)
+	(text "Additional pin functions:\nhttps://pinout.xyz/"
+		(exclude_from_sim no)
+		(at 179.07 180.34 0)
+		(effects
+			(font
+				(size 1.27 1.27)
+			)
+			(justify left bottom)
+		)
 	)
 	(junction
@@
 		)
 	)
-	(text "ID_SD and ID_SC PINS:\nThese pins are reserved for HAT ID EEPROM.\n\nAt boot time this I2C interface will be\ninterrogated to look for an EEPROM\nthat identifes the attached board and\nallows automagic setup of the GPIOs\n(and optionally, Linux drivers).\n\nBridging JP1 enables write protection.\n\nDO NOT USE these pins for anything other\nthan attaching an I2C ID EEPROM. Leave\nunconnected if ID EEPROM not required."
-		(exclude_from_sim no)
-		(at 16.51 193.04 0)
-		(effects
-			(font
-				(size 1.27 1.27)
-			)
-			(justify left bottom)
-		)
-	)
-	(text "Additional pin functions:\nhttps://pinout.xyz/"
-		(exclude_from_sim no)
-		(at 179.07 180.34 0)
-		(effects
-			(font
-				(size 1.27 1.27)
-			)
-			(justify left bottom)
-		)
-	)
 	(label "ID_SDA"
 		(at 31.75 60.96 0)
-		(fields_autoplaced yes)
 		(effects
 			(font
@@
 	(label "GPIO6"
 		(at 31.75 66.04 0)
-		(fields_autoplaced yes)
 		(effects
 			(font
@@
 	(label "ID_SDA"
 		(at 110.49 175.26 180)
-		(fields_autoplaced yes)
 		(effects
 			(font
@@
 	(label "ID_SCL"
 		(at 100.33 60.96 180)
-		(fields_autoplaced yes)
 		(effects
 			(font
@@
 	(label "GPIO5"
 		(at 31.75 63.5 0)
-		(fields_autoplaced yes)
 		(effects
 			(font
@@
 	(label "GPIO21{slash}PCM.DOUT"
 		(at 100.33 76.2 180)
-		(fields_autoplaced yes)
 		(effects
 			(font
@@
 	(label "GPIO19{slash}PCM.FS"
 		(at 31.75 71.12 0)
-		(fields_autoplaced yes)
 		(effects
 			(font
@@
 	(label "GPIO10{slash}SPI0.MOSI"
 		(at 31.75 50.8 0)
-		(fields_autoplaced yes)
 		(effects
 			(font
@@
 	(label "GPIO9{slash}SPI0.MISO"
 		(at 31.75 53.34 0)
-		(fields_autoplaced yes)
 		(effects
 			(font
@@
 	(label "GPIO23"
 		(at 100.33 45.72 180)
-		(fields_autoplaced yes)
 		(effects
 			(font
@@
 	(label "GPIO4{slash}GPCLK0"
 		(at 31.75 35.56 0)
-		(fields_autoplaced yes)
 		(effects
 			(font
@@
 	(label "GPIO27"
 		(at 31.75 43.18 0)
-		(fields_autoplaced yes)
 		(effects
 			(font
@@
 	(label "GPIO26"
 		(at 31.75 73.66 0)
-		(fields_autoplaced yes)
 		(effects
 			(font
@@
 	(label "GPIO14{slash}TXD0"
 		(at 100.33 35.56 180)
-		(fields_autoplaced yes)
 		(effects
 			(font
@@
 	(label "GPIO8{slash}SPI0.CE0"
 		(at 100.33 55.88 180)
-		(fields_autoplaced yes)
 		(effects
 			(font
@@
 	(label "GPIO15{slash}RXD0"
 		(at 100.33 38.1 180)
-		(fields_autoplaced yes)
 		(effects
 			(font
@@
 	(label "GPIO16"
 		(at 100.33 71.12 180)
-		(fields_autoplaced yes)
 		(effects
 			(font
@@
 	(label "GPIO22"
 		(at 31.75 45.72 0)
-		(fields_autoplaced yes)
 		(effects
 			(font
@@
 	(label "GPIO2{slash}SDA1"
 		(at 31.75 30.48 0)
-		(fields_autoplaced yes)
 		(effects
 			(font
@@
 	(label "GPIO17"
 		(at 31.75 40.64 0)
-		(fields_autoplaced yes)
 		(effects
 			(font
@@
 	(label "GPIO25"
 		(at 100.33 53.34 180)
-		(fields_autoplaced yes)
 		(effects
 			(font
@@
 	(label "GPIO3{slash}SCL1"
 		(at 31.75 33.02 0)
-		(fields_autoplaced yes)
 		(effects
 			(font
@@
 	(label "GPIO18{slash}PCM.CLK"
 		(at 100.33 40.64 180)
-		(fields_autoplaced yes)
 		(effects
 			(font
@@
 	(label "GPIO12{slash}PWM0"
 		(at 100.33 66.04 180)
-		(fields_autoplaced yes)
 		(effects
 			(font
@@
 	(label "GPIO13{slash}PWM1"
 		(at 31.75 68.58 0)
-		(fields_autoplaced yes)
 		(effects
 			(font
@@
 	(label "GPIO20{slash}PCM.DIN"
 		(at 100.33 73.66 180)
-		(fields_autoplaced yes)
 		(effects
 			(font
@@
 	(label "GPIO24"
 		(at 100.33 48.26 180)
-		(fields_autoplaced yes)
 		(effects
 			(font
@@
 	(label "GPIO7{slash}SPI0.CE1"
 		(at 100.33 58.42 180)
-		(fields_autoplaced yes)
 		(effects
 			(font
@@
 	(label "ID_SCL"
 		(at 110.49 177.8 180)
-		(fields_autoplaced yes)
 		(effects
 			(font
@@
 	(label "GPIO11{slash}SPI0.SCLK"
 		(at 31.75 55.88 0)
-		(fields_autoplaced yes)
 		(effects
 			(font
@@
 			)
 		)
-		(property "Description" ""
+		(property "Description" "Power symbol creates a global label with name \"+5V\""
 			(at 76.2 24.13 0)
 			(effects
@@
 			)
 		)
-		(property "Description" ""
+		(property "Description" "Power symbol creates a global label with name \"+3.3V\""
 			(at 55.88 24.13 0)
 			(effects
@@
 			)
 		)
-		(property "Description" ""
+		(property "Description" "Power symbol creates a global label with name \"GND\" , ground"
 			(at 76.2 80.01 0)
 			(effects
@@
 			)
 		)
-		(property "Description" ""
+		(property "Description" "Power symbol creates a global label with name \"GND\" , ground"
 			(at 58.42 80.01 0)
 			(effects
@@
 			)
 		)
-		(property "Datasheet" ""
+		(property "Datasheet" "~"
 			(at -57.15 74.93 0)
 			(effects
@@
 			)
 		)
-		(property "Description" ""
+		(property "Description" "Generic connector, double row, 02x20, odd/even pin numbering scheme (row 1 odd numbers, row 2 even numbers), script generated (kicad-library-utils/schlib/autogen/connector/)"
 			(at 66.04 50.8 0)
 			(effects
@@
 			)
 		)
-		(property "Description" ""
+		(property "Description" "Unpolarized capacitor, small symbol"
 			(at 67.31 177.8 0)
 			(effects
@@
 			)
 		)
-		(property "Description" ""
+		(property "Description" "Resistor, small symbol"
 			(at 93.98 170.18 0)
 			(effects
@@
 			)
 		)
-		(property "Description" ""
+		(property "Description" "Solder Jumper, 2-pole, open"
 			(at 96.52 180.34 0)
 			(effects
@@
 			)
 		)
-		(property "Description" ""
+		(property "Description" "Resistor, small symbol"
 			(at 101.6 170.18 0)
 			(effects
@@
 			)
 		)
-		(property "Description" ""
+		(property "Description" "Power symbol creates a global label with name \"+3.3V\""
 			(at 101.6 162.56 0)
 			(effects
@@
 			)
 		)
-		(property "Description" ""
+		(property "Description" "256 kb CMOS Serial EEPROM, DIP-8/SOIC-8/TSSOP-8/DFN-8"
 			(at 81.28 177.8 0)
 			(effects
@@
 			)
 		)
-		(property "Description" ""
+		(property "Description" "Power symbol creates a global label with name \"GND\" , ground"
 			(at 81.28 190.5 0)
 			(effects
@@
 			)
 		)
-		(property "Description" ""
+		(property "Description" "Power symbol creates a global label with name \"+3.3V\""
 			(at 101.6 180.34 0)
 			(effects
@@
 		)
 	)
+	(embedded_fonts no)
 )
