File: Projects/STM32_Nucleo-64_Morpho/STM_Nucleo64_Morpho.kicad_pcb (KiCad board)
At the start: 2 copper layers, 70 x 57.5 mm, 5 parts, among them J1 CN7, J2 CN10

Commit message: feat: update kicad-templates to 9.0.0-1
Signed-off-by: lhdjply <lhdjply@126.com>
Connections:
- J2 pad 7: VDDA -> unconnected-(J2-Pin_7-Pad7)
- J2 pad 9: GND -> unconnected-(J2-Pin_9-Pad9)
